File: Misaka.kicad_pcb (KiCad board)
At the start: 2 copper layers, 100 x 86.6 mm, 104 parts, among them J1 Battery, J2 Conn_01x04_Male, J3 Conn_01x04_Male, J4 Conn_01x04_Male, J5 USB_B_Micro, J6 Conn_01x04_Female, J7 Conn_01x04_Female_UART, J8 Conn_02x04_Odd_Even, J9 Conn_01x07, SW1 SW_DIP_x03, U1 DRV8825PWPR, U2 ATmega2560-16AU, U3 DRV8825PWPR, U4 DRV8825PWPR, U5 CH340C, U6 AMS1117-5.0, U7 AMS1117-3.3, U8 24LC02, Y1 CSTLS16M0X51-B0

Commit message: DEL LED MS123
Parts:
- removed C13: 22pF, Capacitor_SMD:C_0603_1608Metric_Pad1.05x0.95mm_HandSolder
- removed C15, C16: 1uF, Capacitor_SMD:C_0603_1608Metric_Pad1.05x0.95mm_HandSolder
- removed C17, C18, C19, C20, C21, C22, C23, C24: 100nF, Capacitor_SMD:C_0603_1608Metric_Pad1.05x0.95mm_HandSolder
- removed D1: CD1206, Diode_SMD:D_1206_3216Metric_Pad1.42x1.75mm_HandSolder
- removed D10, D3, D4, D5, D6, D7, D8, D9: WS2812B, LED_SMD:LED_WS2812B_PLCC4_5.0x5.0mm_P3.2mm
- removed J8: Conn_02x04_Odd_Even, Connector_PinSocket_1.27mm:PinSocket_2x04_P1.27mm_Vertical
- removed J9: Conn_01x07, Connector_PinSocket_2.54mm:PinSocket_1x07_P2.54mm_Vertical
- removed R28: 1k, Resistor_SMD:R_0603_1608Metric_Pad1.05x0.95mm_HandSolder
- removed R29, R30, R31, R32: 4.7k, Resistor_SMD:R_0603_1608Metric_Pad1.05x0.95mm_HandSolder
- removed S1: TACTILE_SWITCH_SMD_4.5MM, Switches:TACTILE_SWITCH_SMD_4.5MM
- removed SW1: SW_DIP_x03, Button_Switch_SMD:SW_DIP_SPSTx03_Slide_6.7x9.18mm_W8.61mm_P2.54mm_LowProfile
- removed U8: 24LC02, Package_DIP:DIP-8_W7.62mm_Socket_LongPads
- C-VMA1, C-VMA2, C-VMA3, C-VMB1, C-VMB2, C-VMB3, C1, C2, C3, C4, C5, C6, C7, C8, C9, CP1, CP2, CP3, J2, J3, J4, R1, R10, R11, R12, R13, R14, R15, R16, R17, R18, R19, R2, R20, R21, R3, R4, R5, R6, R7, R8, R9, U1, U3, U4: moved to F.Cu
- moved R25 106.3 mm to (123.5, 119.7)
- moved J6 105.9 mm to (143.6, 71.3)
- moved R24 101.2 mm to (123.5, 117.2)
- moved C11 98.6 mm to (115.0, 121.2), turned to 0 degrees
- moved J7 94.0 mm to (110.6, 110.8)
- moved R5 92.2 mm to (129.7, 72.8), turned to 0 degrees
- moved C10 92.0 mm to (110.4, 122.0), turned to 0 degrees
- moved J5 91.7 mm to (125.0, 110.8)
- moved R1 90.6 mm to (129.7, 70.2)
- moved R22 87.8 mm to (123.5, 114.7), turned to 0 degrees
- moved R23 87.7 mm to (127.8, 114.7)
- moved U5 86.9 mm to (117.1, 114.2)
- moved R4 86.5 mm to (125.3, 75.5), turned to 0 degrees
- moved C12 84.8 mm to (127.8, 117.2)
- moved C-VMB1 84.2 mm to (129.6, 75.5), turned to 0 degrees
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Connections:
- J1 pad 1: +12V -> GND
- J1 pad 2: GND -> +12V
- R24 pad 1: /TX0 -> /RX0
- R25 pad 1: /RX0 -> /TX0
- U2 pad 43: /SCL -> (no net)
- U2 pad 44: /SDA -> (no net)
- U2 pad 7: /D3 -> (no net)
Routing:
- net GND: track 647.0 -> 0.00 mm, vias 29 -> 0
- net +5V: track 578.2 -> 0.00 mm, vias 13 -> 0
- net +12V: track 285.8 -> 0.00 mm, vias 11 -> 0
- net +3V3: track 171.9 -> 0.00 mm, vias 4 -> 0
- net /MS3: track 138.4 -> 0.00 mm, vias 9 -> 0
- net /MS2: track 132.7 -> 0.00 mm, vias 8 -> 0
- net /MS1: track 121.8 -> 0.00 mm, vias 7 -> 0
- net /D3: track 89.5 -> 0.00 mm, vias 2 -> 0
- net /D10: track 82.6 -> 0.00 mm, vias 3 -> 0
- net /RESET: track 76.7 -> 0.00 mm, vias 3 -> 0
- net /D9: track 69.9 -> 0.00 mm, vias 3 -> 0
- net /D11: track 69.8 -> 0.00 mm, vias 3 -> 0
- net /D8: track 66.9 -> 0.00 mm, vias 3 -> 0
- net /RX1: track 49.6 -> 0.00 mm
- net /TX1: track 47.4 -> 0.00 mm
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- removed copper zone on B.Cu, net GND
- removed copper zone on F.Cu, net GND
Other:
- board outline removed
