File: Misaka.kicad_pcb (KiCad board)
At the start: 2 copper layers, 74 parts, among them J1 Battery, J2 Conn_01x04_Male, J3 Conn_01x04_Male, J4 Conn_01x04_Male, J5 USB_B_Micro, J6 Conn_01x04_Female, J7 Conn_01x04_Female_UART, U1 DRV8825PWPR, U2 ATmega2560-16AU, U3 DRV8825PWPR, U4 DRV8825PWPR, U5 CH340C, U6 AMS1117-5.0, U7 AMS1117-3.3, Y1 CSTLS16M0X51-B0

Commit message: except GND
Parts:
- removed J7: Conn_01x04_Female_UART, Connector_PinSocket_2.54mm:PinSocket_1x04_P2.54mm_Vertical
- J2, J3, J4: moved to B.Cu
- moved R25 111.5 mm to (25.9, 65.7), turned to 270 degrees
- moved J5 109.5 mm to (21.1, 76.2), turned to 90 degrees
- moved R24 107.2 mm to (29.5, 65.7), turned to 270 degrees
- moved C14 103.8 mm to (108.0, 33.2), turned to 270 degrees
- moved CP4 100.0 mm to (101.9, 28.4)
- moved CP5 99.4 mm to (101.9, 37.3)
- moved J6 99.0 mm to (55.4, 26.4), turned to 270 degrees
- moved C10 97.4 mm to (27.3, 71.1), turned to 180 degrees
- moved U5 88.1 mm to (36.8, 77.7)
- moved C11 87.7 mm to (46.6, 66.3), turned to 180 degrees
- moved C12 85.9 mm to (52.6, 75.8), turned to 180 degrees
- moved R22 83.0 mm to (52.6, 71.5)
- moved R23 82.5 mm to (52.6, 80.8), turned to 180 degrees
- moved RX1 78.4 mm to (34.4, 55.6)
- moved U6 77.4 mm to (90.9, 47.2), turned to 270 degrees
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Connections:
- U1 pad 24: /MS1 -> (no net)
- U1 pad 25: /MS2 -> (no net)
- U1 pad 26: /MS3 -> (no net)
- U3 pad 24: /MS1 -> (no net)
- U3 pad 25: /MS2 -> (no net)
- U3 pad 26: /MS3 -> (no net)
- U4 pad 24: /MS1 -> (no net)
- U4 pad 25: /MS2 -> (no net)
- U4 pad 26: /MS3 -> (no net)
Routing:
- net +5V: track 0.00 -> 325.5 mm, vias 0 -> 5
- net +12V: track 0.00 -> 304.7 mm, vias 0 -> 6
- net /RESET: track 0.00 -> 112.2 mm, vias 0 -> 2
- net +3V3: track 0.00 -> 107.0 mm, vias 0 -> 1
- net /D6: track 0.00 -> 81.4 mm
- net /D7: track 0.00 -> 79.6 mm
- net /RX1: track 0.00 -> 74.8 mm, vias 0 -> 1
- net /TX1: track 0.00 -> 73.7 mm, vias 0 -> 1
- net /D8: track 0.00 -> 54.0 mm
- net /D10: track 0.00 -> 53.9 mm
- net /D11: track 0.00 -> 53.2 mm
- net /D9: track 0.00 -> 52.6 mm
- net /D13: track 0.00 -> 52.4 mm, vias 0 -> 2
- net Net-(C14-Pad1): track 0.00 -> 40.7 mm
- net /RX0: track 0.00 -> 36.5 mm
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Other:
- board outline added: 120 x 103.9 mm

Commit message: Update Misaka.kicad_pcb
Routing:
- net GND: track 8.42 -> 131.8 mm, vias 0 -> 9
- added copper zone on B.Cu, net (none)
- added copper zone on F.Cu, net GND
Changed lines of the file:
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@@
     (thickness 1.6)
     (drawings 9)
-    (tracks 638)
+    (tracks 712)
     (zones 0)
     (modules 73)
@@
   )
   (setup
-    (last_trace_width 0.508)
+    (last_trace_width 0.19)
     (user_trace_width 0.19)
     (user_trace_width 0.254)
@@
   (segment (start 51.55527 36.306921) (end 49.6 34.351651) (width 0.19) (layer F.Cu) (net 6))
   (segment (start 51.556668 36.306921) (end 51.55527 36.306921) (width 0.19) (layer F.Cu) (net 6))
+  (via (at 26.5176 69.09054) (size 0.8) (drill 0.4) (layers F.Cu B.Cu) (net 6))
+  (segment (start 26.444 71.12) (end 26.444 69.16414) (width 0.508) (layer F.Cu) (net 6))
+  (segment (start 26.444 69.16414) (end 26.5176 69.09054) (width 0.508) (layer F.Cu) (net 6))
+  (segment (start 27.083285 69.09054) (end 27.469365 69.47662) (width 0.508) (layer B.Cu) (net 6))
+  (segment (start 26.5176 69.09054) (end 27.083285 69.09054) (width 0.508) (layer B.Cu) (net 6))
+  (segment (start 27.469365 69.47662) (end 33.41116 69.47662) (width 0.508) (layer B.Cu) (net 6))
+  (via (at 34.29762 70.36308) (size 0.8) (drill 0.4) (layers F.Cu B.Cu) (net 6))
+  (segment (start 33.41116 69.47662) (end 34.29762 70.36308) (width 0.508) (layer B.Cu) (net 6))
+  (segment (start 34.29762 73.22162) (end 34.355 73.279) (width 0.508) (layer F.Cu) (net 6))
+  (segment (start 34.29762 70.36308) (end 34.29762 73.22162) (width 0.508) (layer F.Cu) (net 6))
+  (segment (start 83.719 95.091) (end 83.36534 94.73734) (width 0.254) (layer F.Cu) (net 6))
+  (segment (start 83.719 96.266) (end 83.719 95.091) (width 0.254) (layer F.Cu) (net 6))
+  (segment (start 83.36534 94.73734) (end 83.36534 92.6465) (width 0.254) (layer F.Cu) (net 6))
+  (segment (start 84.78 92.436) (end 84.78 91.982) (width 0.254) (layer F.Cu) (net 6))
+  (segment (start 84.5695 92.6465) (end 84.78 92.436) (width 0.254) (layer F.Cu) (net 6))
+  (segment (start 83.36534 92.6465) (end 84.5695 92.6465) (width 0.254) (layer F.Cu) (net 6))
+  (segment (start 89.676 83.532) (end 87.63 85.578) (width 0.254) (layer F.Cu) (net 6))
+  (segment (start 87.63 85.578) (end 87.63 87.757) (width 0.254) (layer F.Cu) (net 6))
+  (segment (start 90.48 83.532) (end 89.676 83.532) (width 0.254) (layer F.Cu) (net 6))
+  (segment (start 87.63 89.936) (end 87.63 87.757) (width 0.254) (layer F.Cu) (net 6))
+  (segment (start 85.584 91.982) (end 87.63 89.936) (width 0.254) (layer F.Cu) (net 6))
+  (segment (start 84.78 91.982) (end 85.584 91.982) (width 0.254) (layer F.Cu) (net 6))
+  (segment (start 87.63 113.431) (end 87.63 111.252) (width 0.254) (layer F.Cu) (net 6))
+  (segment (start 85.584 115.477) (end 87.63 113.431) (width 0.254) (layer F.Cu) (net 6))
+  (segment (start 84.78 115.477) (end 85.584 115.477) (width 0.254) (layer F.Cu) (net 6))
+  (segment (start 87.63 109.073) (end 87.63 111.252) (width 0.254) (layer F.Cu) (net 6))
+  (segment (start 89.676 107.027) (end 87.63 109.073) (width 0.254) (layer F.Cu) (net 6))
+  (segment (start 90.48 107.027) (end 89.676 107.027) (width 0.254) (layer F.Cu) (net 6))
+  (segment (start 87.63 62.083) (end 87.63 64.262) (width 0.254) (layer F.Cu) (net 6))
+  (segment (start 89.676 60.037) (end 87.63 62.083) (width 0.254) (layer F.Cu) (net 6))
+  (segment (start 90.48 60.037) (end 89.676 60.037) (width 0.254) (layer F.Cu) (net 6))
+  (segment (start 87.63 66.441) (end 87.63 64.262) (width 0.254) (layer F.Cu) (net 6))
+  (segment (start 85.584 68.487) (end 87.63 66.441) (width 0.254) (layer F.Cu) (net 6))
+  (segment (start 84.78 68.487) (end 85.584 68.487) (width 0.254) (layer F.Cu) (net 6))
+  (segment (start 83.976 68.487) (end 84.78 68.487) (width 0.254) (layer F.Cu) (net 6))
+  (segment (start 83.117 69.346) (end 83.976 68.487) (width 0.254) (layer F.Cu) (net 6))
+  (segment (start 83.117 72.64) (end 83.117 69.346) (width 0.254) (layer F.Cu) (net 6))
+  (via (at 82.70748 80.69834) (size 0.8) (drill 0.4) (layers F.Cu B.Cu) (net 6))
+  (segment (start 83.453 79.248) (end 83.453 79.95282) (width 0.254) (layer F.Cu) (net 6))
+  (segment (start 83.453 79.95282) (end 82.70748 80.69834) (width 0.254) (layer F.Cu) (net 6))
+  (segment (start 82.70748 80.69834) (end 83.85556 81.84642) (width 0.254) (layer B.Cu) (net 6))
+  (segment (start 87.63 82.753) (end 87.63 87.757) (width 0.254) (layer B.Cu) (net 6))
+  (segment (start 86.72342 81.84642) (end 87.63 82.753) (width 0.254) (layer B.Cu) (net 6))
+  (segment (start 83.85556 81.84642) (end 86.72342 81.84642) (width 0.254) (layer B.Cu) (net 6))
+  (via (at 82.94878 57.00268) (size 0.8) (drill 0.4) (layers F.Cu B.Cu) (net 6))
+  (segment (start 83.34 55.626) (end 83.34 56.61146) (width 0.254) (layer F.Cu) (net 6))
+  (segment (start 83.34 56.61146) (end 82.94878 57.00268) (width 0.254) (layer F.Cu) (net 6))
+  (segment (start 82.94878 57.00268) (end 83.73618 57.79008) (width 0.254) (layer B.Cu) (net 6))
+  (segment (start 87.63 59.258) (end 87.63 64.262) (width 0.254) (layer B.Cu) (net 6))
+  (segment (start 86.16208 57.79008) (end 87.63 59.258) (width 0.254) (layer B.Cu) (net 6))
+  (segment (start 83.73618 57.79008) (end 86.16208 57.79008) (width 0.254) (layer B.Cu) (net 6))
+  (via (at 82.97164 104.50068) (size 0.8) (drill 0.4) (layers F.Cu B.Cu) (net 6))
+  (segment (start 83.34 103.124) (end 83.34 104.13232) (width 0.254) (layer F.Cu) (net 6))
+  (segment (start 83.34 104.13232) (end 82.97164 104.50068) (width 0.254) (layer F.Cu) (net 6))
+  (segment (start 83.537325 104.50068) (end 83.941185 104.90454) (width 0.254) (layer B.Cu) (net 6))
+  (segment (start 82.97164 104.50068) (end 83.537325 104.50068) (width 0.254) (layer B.Cu) (net 6))
+  (segment (start 87.63 106.248) (end 87.63 111.252) (width 0.254) (layer B.Cu) (net 6))
+  (segment (start 86.28654 104.90454) (end 87.63 106.248) (width 0.254) (layer B.Cu) (net 6))
+  (segment (start 83.941185 104.90454) (end 86.28654 104.90454) (width 0.254) (layer B.Cu) (net 6))
+  (segment (start 64.526233 57.647767) (end 64.526233 55.128233) (width 0.254) (layer B.Cu) (net 6))
+  (via (at 63.30696 53.90896) (size 0.8) (drill 0.4) (layers F.Cu B.Cu) (net 6))
+  (segment (start 64.526233 55.128233) (end 63.30696 53.90896) (width 0.254) (layer B.Cu) (net 6))
+  (segment (start 62.2 37.205708) (end 62.2 35.84496) (width 0.254) (layer F.Cu) (net 6))
+  (segment (start 62.2 35.84496) (end 60.11926 33.76422) (width 0.254) (layer F.Cu) (net 6))
+  (via (at 60.11926 33.76422) (size 0.8) (drill 0.4) (layers F.Cu B.Cu) (net 6))
+  (segment (start 49.6 34.351651) (end 47.004549 34.351651) (width 0.254) (layer F.Cu) (net 6))
+  (segment (start 43.121825 38.234375) (end 43.121825 40.6) (width 0.254) (layer F.Cu) (net 6))
+  (segment (start 47.004549 34.351651) (end 43.121825 38.234375) (width 0.254) (layer F.Cu) (net 6))
+  (via (at 46.17466 52.67198) (size 0.8) (drill 0.4) (layers F.Cu B.Cu) (net 6))
+  (segment (start 48.374688 48.911099) (end 46.17466 51.111127) (width 0.19) (layer F.Cu) (net 6))
+  (segment (start 46.17466 51.111127) (end 46.17466 52.67198) (width 0.19) (layer F.Cu) (net 6))
+  (via (at 58.91022 54.74462) (size 0.8) (drill 0.4) (layers F.Cu B.Cu) (net 6))
+  (segment (start 57.796885 51.739526) (end 58.91022 52.852861) (width 0.19) (layer F.Cu) (net 6))
+  (segment (start 58.91022 52.852861) (end 58.91022 54.74462) (width 0.19) (layer F.Cu) (net 6))
   (segment (start 90.588 91.44) (end 90.48 91.332) (width 0.254) (layer F.Cu) (net 7))
   (segment (start 91.44 96.045) (end 92.40201 95.08299) (width 0.254) (layer F.Cu) (net 7))
@@
   (segment (start 33.38 75.819) (end 34.355 75.819) (width 0.254) (layer F.Cu) (net 72))
   (segment (start 25.874 66.621) (end 26.349 66.621) (width 0.254) (layer F.Cu) (net 72))
+  (zone (net 6) (net_name GND) (layer F.Cu) (hatch edge 0.508)
+    (connect_pads (clearance 0.508))
+    (min_thickness 0.254)
+    (fill yes (arc_segments 32) (thermal_gap 0.508) (thermal_bridge_width 0.508))
+    (polygon
+      (pts
+        (xy 134.97814 75.00366) (xy 104.99852 126.95428) (xy 45.01134 126.9365) (xy 15.0114 75.05954) (xy 44.9961 23.04034)
+        (xy 45.00372 23.04034) (xy 104.9909 23.03272)
+      )
+    )
+  )
+  (zone (net 0) (net_name "") (layer B.Cu) (hatch edge 0.508)
+    (connect_pads (clearance 0.508))
+    (min_thickness 0.254)
+    (fill yes (arc_segments 32) (thermal_gap 0.508) (thermal_bridge_width 0.508))
+    (polygon
+      (pts
+        (xy 134.97814 75.00366) (xy 104.99852 126.95428) (xy 45.01134 126.9365) (xy 15.0114 75.05954) (xy 44.9961 23.04034)
+        (xy 45.00372 23.04034) (xy 104.9909 23.03272)
+      )
+    )
+  )
 )

Commit message: gerber
Routing:
- net +5V: track 325.5 -> 326.0 mm
Changed lines of the file:
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@@
     (thickness 1.6)
     (drawings 9)
-    (tracks 712)
+    (tracks 713)
     (zones 0)
     (modules 73)
@@
     (add_net /D10)
     (add_net /D11)
-    (add_net /D12)
     (add_net /D13)
-    (add_net /D3)
-    (add_net /D53)
     (add_net /D6)
     (add_net /D7)
@@
     (add_net /RX1)
     (add_net /RX2)
-    (add_net /RX3)
     (add_net /SCK)
-    (add_net /SCL)
-    (add_net /SDA)
-    (add_net /StepperMotorDriver1/MS1)
-    (add_net /StepperMotorDriver1/MS2)
-    (add_net /StepperMotorDriver1/MS3)
     (add_net /StepperMotorDriver1/V3P3OUT)
-    (add_net /StepperMotorDriver2/MS1)
-    (add_net /StepperMotorDriver2/MS2)
-    (add_net /StepperMotorDriver2/MS3)
     (add_net /StepperMotorDriver2/V3P3OUT)
-    (add_net /StepperMotorDriver3/MS1)
-    (add_net /StepperMotorDriver3/MS2)
-    (add_net /StepperMotorDriver3/MS3)
     (add_net /StepperMotorDriver3/V3P3OUT)
     (add_net /TX0)
     (add_net /TX1)
     (add_net /TX2)
-    (add_net /TX3)
     (add_net "Net-(C1-Pad1)")
     (add_net "Net-(C1-Pad2)")
@@
     (add_net "Net-(J5-Pad2)")
     (add_net "Net-(J5-Pad3)")
-    (add_net "Net-(J5-Pad4)")
     (add_net "Net-(L1-Pad2)")
-    (add_net "Net-(MOD1-Pad11)")
-    (add_net "Net-(MOD1-Pad12)")
-    (add_net "Net-(MOD1-Pad13)")
-    (add_net "Net-(MOD1-Pad14)")
-    (add_net "Net-(MOD1-Pad15)")
-    (add_net "Net-(MOD1-Pad16)")
-    (add_net "Net-(MOD1-Pad17)")
-    (add_net "Net-(MOD1-Pad18)")
-    (add_net "Net-(MOD1-Pad19)")
-    (add_net "Net-(MOD1-Pad20)")
-    (add_net "Net-(MOD1-Pad4)")
-    (add_net "Net-(MOD1-Pad5)")
-    (add_net "Net-(MOD1-Pad6)")
-    (add_net "Net-(MOD1-Pad7)")
-    (add_net "Net-(MOD1-Pad8)")
-    (add_net "Net-(MOD1-Pad9)")
     (add_net "Net-(R11-Pad1)")
     (add_net "Net-(R12-Pad1)")
@@
     (add_net "Net-(R7-Pad1)")
     (add_net "Net-(R8-Pad2)")
-    (add_net "Net-(U1-Pad19)")
-    (add_net "Net-(U1-Pad21)")
-    (add_net "Net-(U1-Pad23)")
-    (add_net "Net-(U2-Pad1)")
-    (add_net "Net-(U2-Pad14)")
-    (add_net "Net-(U2-Pad27)")
-    (add_net "Net-(U2-Pad28)")
-    (add_net "Net-(U2-Pad29)")
-    (add_net "Net-(U2-Pad35)")
-    (add_net "Net-(U2-Pad36)")
-    (add_net "Net-(U2-Pad37)")
-    (add_net "Net-(U2-Pad38)")
-    (add_net "Net-(U2-Pad39)")
-    (add_net "Net-(U2-Pad4)")
-    (add_net "Net-(U2-Pad40)")
-    (add_net "Net-(U2-Pad41)")
-    (add_net "Net-(U2-Pad42)")
-    (add_net "Net-(U2-Pad47)")
-    (add_net "Net-(U2-Pad48)")
-    (add_net "Net-(U2-Pad49)")
-    (add_net "Net-(U2-Pad5)")
-    (add_net "Net-(U2-Pad50)")
-    (add_net "Net-(U2-Pad51)")
-    (add_net "Net-(U2-Pad52)")
-    (add_net "Net-(U2-Pad53)")
-    (add_net "Net-(U2-Pad54)")
-    (add_net "Net-(U2-Pad55)")
-    (add_net "Net-(U2-Pad56)")
-    (add_net "Net-(U2-Pad57)")
-    (add_net "Net-(U2-Pad58)")
-    (add_net "Net-(U2-Pad59)")
-    (add_net "Net-(U2-Pad6)")
-    (add_net "Net-(U2-Pad60)")
-    (add_net "Net-(U2-Pad65)")
-    (add_net "Net-(U2-Pad66)")
-    (add_net "Net-(U2-Pad67)")
-    (add_net "Net-(U2-Pad68)")
-    (add_net "Net-(U2-Pad69)")
-    (add_net "Net-(U2-Pad70)")
-    (add_net "Net-(U2-Pad71)")
-    (add_net "Net-(U2-Pad72)")
-    (add_net "Net-(U2-Pad73)")
-    (add_net "Net-(U2-Pad74)")
-    (add_net "Net-(U2-Pad75)")
-    (add_net "Net-(U2-Pad76)")
-    (add_net "Net-(U2-Pad77)")
-    (add_net "Net-(U2-Pad78)")
-    (add_net "Net-(U2-Pad79)")
-    (add_net "Net-(U2-Pad8)")
-    (add_net "Net-(U2-Pad82)")
-    (add_net "Net-(U2-Pad83)")
-    (add_net "Net-(U2-Pad84)")
-    (add_net "Net-(U2-Pad85)")
-    (add_net "Net-(U2-Pad86)")
-    (add_net "Net-(U2-Pad87)")
-    (add_net "Net-(U2-Pad88)")
-    (add_net "Net-(U2-Pad89)")
-    (add_net "Net-(U2-Pad9)")
-    (add_net "Net-(U2-Pad90)")
-    (add_net "Net-(U2-Pad91)")
-    (add_net "Net-(U2-Pad92)")
-    (add_net "Net-(U2-Pad93)")
-    (add_net "Net-(U2-Pad94)")
-    (add_net "Net-(U2-Pad95)")
-    (add_net "Net-(U2-Pad96)")
-    (add_net "Net-(U2-Pad97)")
-    (add_net "Net-(U2-Pad98)")
-    (add_net "Net-(U3-Pad19)")
-    (add_net "Net-(U3-Pad21)")
-    (add_net "Net-(U3-Pad23)")
-    (add_net "Net-(U4-Pad19)")
-    (add_net "Net-(U4-Pad21)")
-    (add_net "Net-(U4-Pad23)")
-    (add_net "Net-(U5-Pad10)")
-    (add_net "Net-(U5-Pad11)")
-    (add_net "Net-(U5-Pad12)")
-    (add_net "Net-(U5-Pad14)")
-    (add_net "Net-(U5-Pad15)")
-    (add_net "Net-(U5-Pad7)")
-    (add_net "Net-(U5-Pad8)")
-    (add_net "Net-(U5-Pad9)")
   )
   (net_class Power ""
@@
   (segment (start 48.019735 48.557546) (end 41.261 55.316281) (width 0.19) (layer F.Cu) (net 16))
   (segment (start 48.021134 48.557546) (end 48.019735 48.557546) (width 0.19) (layer F.Cu) (net 16))
-  (segment (start 55.43 27.44) (end 55.43 26.4) (width 0.19) (layer F.Cu) (net 16))
-  (segment (start 51.318274 31.551726) (end 55.43 27.44) (width 0.19) (layer F.Cu) (net 16))
-  (segment (start 51.318274 35.36142) (end 51.318274 31.551726) (width 0.19) (layer F.Cu) (net 16))
-  (segment (start 51.910221 35.953367) (end 51.318274 35.36142) (width 0.19) (layer F.Cu) (net 16))
   (segment (start 68.001001 27.361001) (end 67.651999 27.011999) (width 0.19) (layer F.Cu) (net 16))
   (segment (start 68.001001 32.114611) (end 68.001001 27.361001) (width 0.19) (layer F.Cu) (net 16))
@@
   (segment (start 96.774 46.96) (end 93.34 50.394) (width 0.508) (layer F.Cu) (net 16))
   (segment (start 96.774 42.164) (end 96.774 46.96) (width 0.508) (layer F.Cu) (net 16))
+  (segment (start 55.43 27.44) (end 55.43 26.4) (width 0.19) (layer F.Cu) (net 16))
+  (segment (start 50.66284 32.20716) (end 55.43 27.44) (width 0.19) (layer F.Cu) (net 16))
+  (segment (start 50.66284 34.707385) (end 50.66284 32.20716) (width 0.19) (layer F.Cu) (net 16))
+  (segment (start 51.910221 35.953367) (end 51.908822 35.953367) (width 0.19) (layer F.Cu) (net 16))
+  (segment (start 51.908822 35.953367) (end 50.66284 34.707385) (width 0.19) (layer F.Cu) (net 16))
   (segment (start 39.605 76.789) (end 51.165666 76.789) (width 0.508) (layer F.Cu) (net 17))
   (segment (start 51.703 76.251666) (end 51.703 75.776666) (width 0.508) (layer F.Cu) (net 17))
