File: Misaka.kicad_pcb (KiCad board)
At the start: 2 copper layers, 120 x 103.9 mm, 73 parts, among them J1 Battery, J2 Conn_01x04_Male, J3 Conn_01x04_Male, J4 Conn_01x04_Male, J5 USB_B_Micro, J6 Conn_01x04_Female, U1 DRV8825PWPR, U2 ATmega2560-16AU, U3 DRV8825PWPR, U4 DRV8825PWPR, U5 CH340C, U6 AMS1117-5.0, U7 AMS1117-3.3, Y1 CSTLS16M0X51-B0

Commit message: v3.1
Parts:
- added C13: 22pF, Capacitor_SMD:C_0603_1608Metric_Pad1.05x0.95mm_HandSolder, F.Cu at (62.7, 90.8)
- added L2: LED, LED_SMD:LED_0603_1608Metric_Pad1.05x0.95mm_HandSolder, F.Cu at (26.7, 88.2)
- added R27: 1k, Resistor_SMD:R_0603_1608Metric_Pad1.05x0.95mm_HandSolder, F.Cu at (32.2, 88.2)
- added RESET1: SW_Push, Button_Switch_SMD:SW_SPST_TL3305A, F.Cu at (62.7, 79.9)
Routing:
- net /RESET: track 112.2 -> 142.2 mm
- net GND: track 131.8 -> 139.3 mm
- net +5V: track 326.0 -> 331.7 mm
- net Net-(L2-Pad2): track 0.00 -> 3.75 mm
