File: Indicator.sch (KiCad schematic (older format))
At the start: 6 parts

Commit message: v3.1
Parts:
- added L2: LED, LED_SMD:LED_0603_1608Metric_Pad1.05x0.95mm_HandSolder, symbol Device:LED
- added R27: 1k, Resistor_SMD:R_0603_1608Metric_Pad1.05x0.95mm_HandSolder, symbol Device:R
Connections:
- net +5V: now also R27.2
- net GND: now also L2.1 (K)
- new net: L2.2 (A), R27.1
Changed lines of the file:
@@
 	1    0    0    -1
 $EndComp
+$Comp
+L Device:R R27
+U 1 1 5E92D40A
+P 2900 3100
+F 0 "R27" V 2693 3100 50  0000 C CNN
+F 1 "1k" V 2784 3100 50  0000 C CNN
+F 2 "Resistor_SMD:R_0603_1608Metric_Pad1.05x0.95mm_HandSolder" V 2830 3100 50  0001 C CNN
+F 3 "~" H 2900 3100 50  0001 C CNN
+	1    2900 3100
+	0    1    1    0
+$EndComp
+$Comp
+L Device:LED L2
+U 1 1 5E92DD88
+P 3350 3100
+F 0 "L2" H 3343 2845 50  0000 C CNN
+F 1 "LED" H 3343 2936 50  0000 C CNN
+F 2 "LED_SMD:LED_0603_1608Metric_Pad1.05x0.95mm_HandSolder" H 3350 3100 50  0001 C CNN
+F 3 "~" H 3350 3100 50  0001 C CNN
+	1    3350 3100
+	-1   0    0    1
+$EndComp
+$Comp
+L power:GND #PWR0113
+U 1 1 5E92E6A3
+P 3650 3100
+F 0 "#PWR0113" H 3650 2850 50  0001 C CNN
+F 1 "GND" H 3655 2927 50  0000 C CNN
+F 2 "" H 3650 3100 50  0001 C CNN
+F 3 "" H 3650 3100 50  0001 C CNN
+	1    3650 3100
+	1    0    0    -1
+$EndComp
+$Comp
+L power:+5V #PWR0157
+U 1 1 5E92ECB8
+P 2600 2950
+F 0 "#PWR0157" H 2600 2800 50  0001 C CNN
+F 1 "+5V" H 2615 3123 50  0000 C CNN
+F 2 "" H 2600 2950 50  0001 C CNN
+F 3 "" H 2600 2950 50  0001 C CNN
+	1    2600 2950
+	1    0    0    -1
+$EndComp
+Wire Wire Line
+	2600 2950 2600 3100
+Wire Wire Line
+	2600 3100 2750 3100
+Wire Wire Line
+	3050 3100 3200 3100
+Wire Wire Line
+	3500 3100 3650 3100
 $EndSCHEMATC
